File: templates/default/default.kicad_pcb (KiCad board)
At the start: 2 copper layers, 0 parts

Commit message: updated default PCB template file
Other:
- board outline added: 80 x 60 mm
Changed lines of the file:
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@@
 	)
 	(net 0 "")
+	(gr_rect
+		(start 110 70)
+		(end 190 130)
+		(stroke
+			(width 0.1)
+			(type default)
+		)
+		(fill no)
+		(layer "Edge.Cuts")
+	)
 	(embedded_fonts no)
 )
