File: projects/lib_test/potentiometers/potentiometers.kicad_sch (KiCad schematic)
At the start: 3 parts, among them P1001 500R, P1002 2k, P1003 5k

Commit message: updated potentiometers test project
Other:
- title: Project name -> Potentiometers
Changed lines of the file:
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@@
 	(paper "A4")
 	(title_block
-		(title "Project name")
-		(date "2025-05-26")
+		(title "Potentiometers")
+		(date "2026-01-10")
 		(rev "1")
-		(comment 1 "PCA number")
-		(comment 2 "PCB number")
+		(comment 1 "-")
+		(comment 2 "-")
 	)
 	(symbol
