File: projects/lib_test/integrated_circuits/adc_dac.kicad_sch (KiCad schematic)
At the start: 1 part, among them U4001 DAC7311

Commit message: updated test projects
Parts:
- renumbered U4001 to U1005
Changed lines of the file:
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@@
 		(on_board yes)
 		(dnp no)
-		(property "Reference" "U4001"
+		(property "Reference" "U1005"
 			(at 40.64 24.13 0)
 			(effects
@@
 			(project ""
 				(path "/e63e39d7-6ac0-4ffd-8aa3-1841a4541b55/55b71c63-df37-48d7-8aea-a12a2b7d7120"
-					(reference "U4001")
+					(reference "U1005")
 					(unit 1)
 				)
