File: projects/lib_test/integrated_circuits/opamps.kicad_sch (KiCad schematic)
At the start: 2 parts, among them U11001 MCP6022, U11002 TLV272

Commit message: updated ic test project
Changed lines of the file:
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@@
 	(title_block
 		(title "Integrated circuits")
-		(date "2026-01-06")
+		(date "2026-01-10")
 		(rev "1")
 		(comment 1 "-")
@@
 		(dnp no)
 		(property "Reference" "U11002"
-			(at 156.21 29.21 0)
+			(at 154.94 15.24 0)
 			(effects
 				(font
@@
 		)
 		(property "Value" "TLV272"
-			(at 156.21 31.75 0)
+			(at 154.94 17.78 0)
 			(effects
 				(font
@@
 		(dnp no)
 		(property "Reference" "U11001"
-			(at 80.01 29.21 0)
+			(at 78.74 15.24 0)
 			(effects
 				(font
@@
 		)
 		(property "Value" "MCP6022"
-			(at 80.01 31.75 0)
-			(effects
-				(font
+			(at 78.74 17.78 0)
+			(effects
+				(font

Commit message: updated test projects
Parts:
- renumbered U11001 to U1030, U11002 to U1031
Changed lines of the file:
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@@
 		(on_board yes)
 		(dnp no)
-		(property "Reference" "U11002"
+		(property "Reference" "U1031"
 			(at 154.94 15.24 0)
 			(effects
@@
 			(project ""
 				(path "/e63e39d7-6ac0-4ffd-8aa3-1841a4541b55/bd7fe9ed-ddb9-415a-abb3-6877f614ff8c"
-					(reference "U11002")
+					(reference "U1031")
 					(unit 3)
 				)
@@
 		(on_board yes)
 		(dnp no)
-		(property "Reference" "U11002"
+		(property "Reference" "U1031"
 			(at 129.54 22.86 0)
 			(effects
@@
 			(project ""
 				(path "/e63e39d7-6ac0-4ffd-8aa3-1841a4541b55/bd7fe9ed-ddb9-415a-abb3-6877f614ff8c"
-					(reference "U11002")
+					(reference "U1031")
 					(unit 2)
 				)
@@
 		(on_board yes)
 		(dnp no)
-		(property "Reference" "U11002"
+		(property "Reference" "U1031"
 			(at 104.14 22.86 0)
 			(effects
@@
 			(project ""
 				(path "/e63e39d7-6ac0-4ffd-8aa3-1841a4541b55/bd7fe9ed-ddb9-415a-abb3-6877f614ff8c"
-					(reference "U11002")
+					(reference "U1031")
 					(unit 1)
 				)
@@
 		(on_board yes)
 		(dnp no)
-		(property "Reference" "U11001"
+		(property "Reference" "U1030"
 			(at 27.94 22.86 0)
 			(effects
@@
 			(project ""
 				(path "/e63e39d7-6ac0-4ffd-8aa3-1841a4541b55/bd7fe9ed-ddb9-415a-abb3-6877f614ff8c"
-					(reference "U11001")
+					(reference "U1030")
 					(unit 1)
 				)
@@
 		(on_board yes)
 		(dnp no)
-		(property "Reference" "U11001"
+		(property "Reference" "U1030"
 			(at 53.34 22.86 0)
 			(effects
@@
 			(project ""
 				(path "/e63e39d7-6ac0-4ffd-8aa3-1841a4541b55/bd7fe9ed-ddb9-415a-abb3-6877f614ff8c"
-					(reference "U11001")
+					(reference "U1030")
 					(unit 2)
 				)
@@
 		(on_board yes)
 		(dnp no)
-		(property "Reference" "U11001"
+		(property "Reference" "U1030"
 			(at 78.74 15.24 0)
 			(effects
@@
 			(project ""
 				(path "/e63e39d7-6ac0-4ffd-8aa3-1841a4541b55/bd7fe9ed-ddb9-415a-abb3-6877f614ff8c"
-					(reference "U11001")
+					(reference "U1030")
 					(unit 3)
 				)
