File: projects/lib_test/integrated_circuits/timers.kicad_sch (KiCad schematic)
At the start: 1 part, among them U12001 NE555

Commit message: updated test projects
Parts:
- renumbered U12001 to U1032
Changed lines of the file:
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@@
 		(on_board yes)
 		(dnp no)
-		(property "Reference" "U12001"
+		(property "Reference" "U1032"
 			(at 43.18 24.13 0)
 			(effects
@@
 			(project ""
 				(path "/e63e39d7-6ac0-4ffd-8aa3-1841a4541b55/da1ff43c-dafd-4fdb-b10c-4c2ad42bbb42"
-					(reference "U12001")
+					(reference "U1032")
 					(unit 1)
 				)
