File: projects/lib_test/integrated_circuits/voltage_regulators.kicad_sch (KiCad schematic)
At the start: 8 parts, among them U10001 REF3040, U10002 AP2120N-3.3, U10003 AP62200, U10004 AZ1117C, U10005 LM317, U10006 LM337, U10007 TPS5430, U10008 TPS82130

Commit message: updated ic test project
Parts:
- renumbered U10004 to U10003, U10003 to U10004, U10007 to U10005, U10008 to U10006, U10005 to U10007, U10006 to U10008
Changed lines of the file:
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@@
 	(title_block
 		(title "Integrated circuits")
-		(date "2026-01-06")
+		(date "2026-01-10")
 		(rev "1")
 		(comment 1 "-")
@@
 		(on_board yes)
 		(dnp no)
-		(property "Reference" "U10004"
+		(property "Reference" "U10003"
 			(at 106.68 20.32 0)
 			(effects
@@
 			(project ""
 				(path "/e63e39d7-6ac0-4ffd-8aa3-1841a4541b55/aab8d68a-9445-4e01-a879-d4613f75fbd3"
-					(reference "U10004")
+					(reference "U10003")
 					(unit 1)
 				)
@@
 		(on_board yes)
 		(dnp no)
-		(property "Reference" "U10006"
+		(property "Reference" "U10008"
 			(at 69.85 63.5 0)
 			(effects
@@
 			(project ""
 				(path "/e63e39d7-6ac0-4ffd-8aa3-1841a4541b55/aab8d68a-9445-4e01-a879-d4613f75fbd3"
-					(reference "U10006")
+					(reference "U10008")
 					(unit 1)
 				)
@@
 		(on_board yes)
 		(dnp no)
-		(property "Reference" "U10003"
+		(property "Reference" "U10004"
 			(at 144.78 20.32 0)
 			(effects
@@
 			(project ""
 				(path "/e63e39d7-6ac0-4ffd-8aa3-1841a4541b55/aab8d68a-9445-4e01-a879-d4613f75fbd3"
-					(reference "U10003")
+					(reference "U10004")
 					(unit 1)
 				)
@@
 		(on_board yes)
 		(dnp no)
-		(property "Reference" "U10005"
+		(property "Reference" "U10007"
 			(at 31.75 43.18 0)
 			(effects
@@
 			(project ""
 				(path "/e63e39d7-6ac0-4ffd-8aa3-1841a4541b55/aab8d68a-9445-4e01-a879-d4613f75fbd3"
-					(reference "U10005")
+					(reference "U10007")
 					(unit 1)
 				)
@@
 		(on_board yes)
 		(dnp no)
-		(property "Reference" "U10007"
+		(property "Reference" "U10005"
 			(at 195.58 20.32 0)
 			(effects
@@
 			(project ""
 				(path "/e63e39d7-6ac0-4ffd-8aa3-1841a4541b55/aab8d68a-9445-4e01-a879-d4613f75fbd3"
-					(reference "U10007")
+					(reference "U10005")
 					(unit 1)
 				)
@@
 		(on_board yes)
 		(dnp no)
-		(property "Reference" "U10008"
+		(property "Reference" "U10006"
 			(at 246.38 20.32 0)
 			(effects
@@
 			(project ""
 				(path "/e63e39d7-6ac0-4ffd-8aa3-1841a4541b55/aab8d68a-9445-4e01-a879-d4613f75fbd3"
-					(reference "U10008")
+					(reference "U10006")
 					(unit 1)
 				)

Commit message: updated test projects
Parts:
- renumbered U10001 to U1022, U10002 to U1023, U10003 to U1024, U10004 to U1025, U10005 to U1026, U10006 to U1027, U10007 to U1028, U10008 to U1029
Changed lines of the file:
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@@
 		(on_board yes)
 		(dnp no)
-		(property "Reference" "U10001"
+		(property "Reference" "U1022"
 			(at 30.48 20.32 0)
 			(effects
@@
 			(project ""
 				(path "/e63e39d7-6ac0-4ffd-8aa3-1841a4541b55/aab8d68a-9445-4e01-a879-d4613f75fbd3"
-					(reference "U10001")
+					(reference "U1022")
 					(unit 1)
 				)
@@
 		(on_board yes)
 		(dnp no)
-		(property "Reference" "U10003"
+		(property "Reference" "U1024"
 			(at 106.68 20.32 0)
 			(effects
@@
 			(project ""
 				(path "/e63e39d7-6ac0-4ffd-8aa3-1841a4541b55/aab8d68a-9445-4e01-a879-d4613f75fbd3"
-					(reference "U10003")
+					(reference "U1024")
 					(unit 1)
 				)
@@
 		(on_board yes)
 		(dnp no)
-		(property "Reference" "U10008"
+		(property "Reference" "U1029"
 			(at 69.85 63.5 0)
 			(effects
@@
 			(project ""
 				(path "/e63e39d7-6ac0-4ffd-8aa3-1841a4541b55/aab8d68a-9445-4e01-a879-d4613f75fbd3"
-					(reference "U10008")
+					(reference "U1029")
 					(unit 1)
 				)
@@
 		(on_board yes)
 		(dnp no)
-		(property "Reference" "U10004"
+		(property "Reference" "U1025"
 			(at 144.78 20.32 0)
 			(effects
@@
 			(project ""
 				(path "/e63e39d7-6ac0-4ffd-8aa3-1841a4541b55/aab8d68a-9445-4e01-a879-d4613f75fbd3"
-					(reference "U10004")
+					(reference "U1025")
 					(unit 1)
 				)
@@
 		(on_board yes)
 		(dnp no)
-		(property "Reference" "U10002"
+		(property "Reference" "U1023"
 			(at 66.04 20.32 0)
 			(effects
@@
 			(project ""
 				(path "/e63e39d7-6ac0-4ffd-8aa3-1841a4541b55/aab8d68a-9445-4e01-a879-d4613f75fbd3"
-					(reference "U10002")
+					(reference "U1023")
 					(unit 1)
 				)
@@
 		(on_board yes)
 		(dnp no)
-		(property "Reference" "U10007"
+		(property "Reference" "U1028"
 			(at 31.75 43.18 0)
 			(effects
@@
 			(project ""
 				(path "/e63e39d7-6ac0-4ffd-8aa3-1841a4541b55/aab8d68a-9445-4e01-a879-d4613f75fbd3"
-					(reference "U10007")
+					(reference "U1028")
 					(unit 1)
 				)
@@
 		(on_board yes)
 		(dnp no)
-		(property "Reference" "U10005"
+		(property "Reference" "U1026"
 			(at 195.58 20.32 0)
 			(effects
@@
 			(project ""
 				(path "/e63e39d7-6ac0-4ffd-8aa3-1841a4541b55/aab8d68a-9445-4e01-a879-d4613f75fbd3"
-					(reference "U10005")
+					(reference "U1026")
 					(unit 1)
 				)
@@
 		(on_board yes)
 		(dnp no)
-		(property "Reference" "U10006"
+		(property "Reference" "U1027"
 			(at 246.38 20.32 0)
 			(effects
@@
 			(project ""
 				(path "/e63e39d7-6ac0-4ffd-8aa3-1841a4541b55/aab8d68a-9445-4e01-a879-d4613f75fbd3"
-					(reference "U10006")
+					(reference "U1027")
 					(unit 1)
 				)
