File: projects/lib_test/integrated_circuits/voltage_regulators.kicad_sch (KiCad schematic)
At the start: 8 parts, among them U1022 REF3040, U1023 AP2120N-3.3, U1024 AZ1117C, U1025 AP62200, U1026 TPS5430, U1027 TPS82130, U1028 LM317, U1029 LM337

Commit message: add AP2205 LDO regulator
Parts:
- added U1035: AP2205, lily_footprints:sot23-5, symbol lily_symbols:ic_volt_reg_AP2205_sot23-5
