File: projects/lib_test/integrated_circuits/integrated_circuits.kicad_pcb (KiCad board)
At the start: 2 copper layers, 70 x 79 mm, 34 parts, among them U1001 ZXCT1010, U1002 LM335, U1003 ADXL345, U1004 LM393, U1005 DAC7311, U1006 93LC56B, U1007 MX25L3233F, U1008 XC7A35T-XCSG325, U1009 TXB0104, U1010 SN75176B, U1011 TUSB4041I, U1012 FT2232HL, U1013 FT2232HQ, U1014 FT231XS, U1015 ESP32-C3FH4, U1016 ATMEGA32A, U1017 ATMEGA168PB, U1018 ATMEGA328PB, U1019 ESP32-C3-MINI-1, U1020 ESP32-C6-MINI-1, U1021 RFM95W-868S2, U1022 REF3040, U1023 AP2120N-3.3, U1024 AZ1117C, U1025 AP62200, U1026 TPS5430, U1027 TPS82130, U1028 LM317, U1029 LM337, U1030 MCP6022, U1031 TLV272, U1032 NE555, U1033 BQ24073, U1034 AT24QT1010

Commit message: add AP2205 LDO regulator
Parts:
- added U1035: AP2205, lily_footprints:sot23-5, F.Cu at (131.0, 116.0)
