File: projects/lib_test/connectors/connectors.kicad_pcb (KiCad board)
At the start: 2 copper layers, 213 x 104 mm, 29 parts, among them X1001 1x02_PH, X1002 1x02_VH, X1003 1x02_PH, X1004 1x06_PH, X1005 1x07_PH, X1006 1x08_PH, X1007 1x06, X1008 1x10, X1009 2x03, X1010 1x15, X1011 2p_5.08, X1012 socket_male, X1013 3p_5.08, X1014 1x03_PH, X1015 1x03_PH, X1016 1x04_PH, X1017 1x04_VH, X1018 1x04_PH, X1019 din41612_plug, X1020 din41612_receptacle, X1021 din41612_receptacle, X1022 dc_005, X1023 sub_d_hd_plug, X1024 sub_d_hd_receptacle, X1025 usb_c, X1026 usb_b, X1027 SMA, X1028 RCJ6A-H, X1029 TC2030-IDC

Commit message: add header 2 pin 5.08mm pitch
Parts:
- added X1017: 1x02, lily_footprints:con_header_1x02_5.08mm_th, F.Cu at (165.0, 147.0)
- renumbered X1019 to X1001, X1001 to X1002, X1014 to X1003, X1016 to X1004, X1002 to X1005, X1015 to X1006, X1017 to X1007, X1020 to X1008, X1003 to X1009, X1018 to X1010, X1004 to X1011, X1021 to X1012, X1005 to X1013, X1006 to X1014, X1023 to X1015, X1007 to X1016, X1008 to X1018, X1024 to X1019, X1009 to X1020, X1010 to X1021, X1011 to X1022, X1013 to X1023, X1012 to X1024, X1028 to X1027, X1029 to X1028, X1022 to X1029, X1027 to X1030

Commit message: add jumper to project
Parts:
- added X1031: 1x02, lily_footprints:con_header_1x02_2.54mm_th, F.Cu at (209.3, 117.0)
