File: test_projects/lib_test/design_blocks/design_blocks.kicad_pcb (KiCad board)
At the start: 2 copper layers, 19 parts, among them U2001 FT231XS, X2001 usb_c

Commit message: update pcb
Other:
- board outline added: 60 x 40 mm
