File: test_projects/lib_test/crystals/crystals.kicad_sch (KiCad schematic)
At the start: 3 parts, among them X1001 12MHz, X1002 16MHz, X1003 50MHz

Commit message: updated Lily IDs
Parts:
- X1001: Lily_ID NO_ID -> 1917-10001
- X1002: Lily_ID NO_ID -> 1917-10002
- X1003: Lily_ID NO_ID -> 1917-10003
