File: test_projects/lib_test/inductors/inductors.kicad_sch (KiCad schematic)
At the start: 4 parts

Commit message: updated Lily IDs
Parts:
- L1001: Lily_ID NO_ID -> 1916-10001
- L1002: Lily_ID NO_ID -> 1916-10002
- L1003: Lily_ID NO_ID -> 1916-10003
- L1004: Lily_ID NO_ID -> 1916-10004
