File: test_projects/lib_test/integrated_circuits/adc_dac.kicad_sch (KiCad schematic)
At the start: 1 part, among them U1005 DAC7311

Commit message: updated Lily IDs
Parts:
- U1005: Lily_ID NO_ID -> 1914-10005
Changed lines of the file:
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@@
 			)
 		)
-		(property "Lily_ID" "NO_ID"
+		(property "Lily_ID" "1914-10005"
 			(at 38.1 76.2 0)
 			(hide yes)
