File: test_projects/lib_test/integrated_circuits/battery_chargers.kicad_sch (KiCad schematic)
At the start: 1 part, among them U1033 BQ24073

Commit message: updated Lily IDs
Parts:
- U1033: Lily_ID NO_ID -> 1914-10002
Changed lines of the file:
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@@
 			)
 		)
-		(property "Lily_ID" "NO_ID"
+		(property "Lily_ID" "1914-10002"
 			(at 40.64 88.9 0)
 			(hide yes)
