File: test_projects/lib_test/integrated_circuits/interfaces.kicad_sch (KiCad schematic)
At the start: 6 parts, among them U1009 TXB0104, U1010 SN75176B, U1011 TUSB4041I, U1012 FT2232HL, U1013 FT2232HQ, U1014 FT231XS

Commit message: updated Lily IDs
Parts:
- U1009: Lily_ID NO_ID -> 1914-10009
- U1010: Lily_ID NO_ID -> 1914-10022
- U1011: Lily_ID NO_ID -> 1914-10023
- U1012: Lily_ID NO_ID -> 1914-10024
- U1013: Lily_ID NO_ID -> 1914-10025
- U1014: Lily_ID NO_ID -> 1914-10026
Changed lines of the file:
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@@
 			)
 		)
-		(property "Lily_ID" "NO_ID"
+		(property "Lily_ID" "1914-10023"
 			(at 243.84 147.32 0)
 			(hide yes)
@@
 			)
 		)
-		(property "Lily_ID" "NO_ID"
+		(property "Lily_ID" "1914-10009"
 			(at 35.56 81.28 0)
 			(hide yes)
@@
 			)
 		)
-		(property "Lily_ID" "NO_ID"
+		(property "Lily_ID" "1914-10024"
 			(at 121.92 170.18 0)
 			(hide yes)
@@
 			)
 		)
-		(property "Lily_ID" "NO_ID"
+		(property "Lily_ID" "1914-10026"
 			(at 43.18 144.78 0)
 			(hide yes)
@@
 			)
 		)
-		(property "Lily_ID" "NO_ID"
+		(property "Lily_ID" "1914-10025"
 			(at 182.88 170.18 0)
 			(hide yes)
@@
 			)
 		)
-		(property "Lily_ID" "NO_ID"
+		(property "Lily_ID" "1914-10022"
 			(at 73.66 81.28 0)
 			(hide yes)
