File: test_projects/lib_test/integrated_circuits/microcontrollers.kicad_sch (KiCad schematic)
At the start: 4 parts, among them U1015 ESP32-C3FH4, U1016 ATMEGA32A, U1017 ATMEGA168PB, U1018 ATMEGA328PB

Commit message: updated Lily IDs
Parts:
- U1015: Lily_ID NO_ID -> 1914-10013
- U1016: Lily_ID NO_ID -> 1914-10012
- U1017: Lily_ID NO_ID -> 1914-10010
- U1018: Lily_ID NO_ID -> 1914-10011
Changed lines of the file:
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@@
 			)
 		)
-		(property "Lily_ID" "NO_ID"
+		(property "Lily_ID" "1914-10013"
 			(at 203.2 139.7 0)
 			(hide yes)
@@
 			)
 		)
-		(property "Lily_ID" "NO_ID"
+		(property "Lily_ID" "1914-10010"
 			(at 91.44 109.22 0)
 			(hide yes)
@@
 			)
 		)
-		(property "Lily_ID" "NO_ID"
+		(property "Lily_ID" "1914-10011"
 			(at 142.24 111.76 0)
 			(hide yes)
@@
 			)
 		)
-		(property "Lily_ID" "NO_ID"
+		(property "Lily_ID" "1914-10012"
 			(at 41.91 124.46 0)
 			(hide yes)
