File: test_projects/lib_test/integrated_circuits/opamps.kicad_sch (KiCad schematic)
At the start: 2 parts, among them U1030 MCP6022, U1031 TLV272

Commit message: updated Lily IDs
Parts:
- U1030: Lily_ID NO_ID -> 1914-10017
- U1031: Lily_ID NO_ID -> 1914-10018
Changed lines of the file:
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@@
 			)
 		)
-		(property "Lily_ID" "NO_ID"
+		(property "Lily_ID" "1914-10018"
 			(at 160.02 45.72 0)
 			(hide yes)
@@
 			)
 		)
-		(property "Lily_ID" "NO_ID"
+		(property "Lily_ID" "1914-10018"
 			(at 134.62 53.34 0)
 			(hide yes)
@@
 			)
 		)
-		(property "Lily_ID" "NO_ID"
+		(property "Lily_ID" "1914-10018"
 			(at 109.22 53.34 0)
 			(hide yes)
@@
 			)
 		)
-		(property "Lily_ID" "NO_ID"
+		(property "Lily_ID" "1914-10017"
 			(at 33.02 53.34 0)
 			(hide yes)
@@
 			)
 		)
-		(property "Lily_ID" "NO_ID"
+		(property "Lily_ID" "1914-10017"
 			(at 58.42 53.34 0)
 			(hide yes)
@@
 			)
 		)
-		(property "Lily_ID" "NO_ID"
+		(property "Lily_ID" "1914-10017"
 			(at 83.82 45.72 0)
 			(hide yes)
