File: test_projects/lib_test/integrated_circuits/sensors.kicad_sch (KiCad schematic)
At the start: 4 parts, among them U1001 ZXCT1010, U1002 LM335, U1003 ADXL345, U1034 AT24QT1010

Commit message: updated Lily IDs
Parts:
- U1001: Lily_ID NO_ID -> 1914-10004
- U1002: Lily_ID NO_ID -> 1914-10019
- U1003: Lily_ID NO_ID -> 1914-10001
- U1034: Lily_ID NO_ID -> 1914-10021
Changed lines of the file:
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@@
 			)
 		)
-		(property "Lily_ID" "NO_ID"
+		(property "Lily_ID" "1914-10001"
 			(at 38.1 83.82 0)
 			(hide yes)
@@
 			)
 		)
-		(property "Lily_ID" "NO_ID"
+		(property "Lily_ID" "1914-10019"
 			(at 127 55.88 0)
 			(hide yes)
@@
 			)
 		)
-		(property "Lily_ID" "NO_ID"
+		(property "Lily_ID" "1914-10021"
 			(at 160.02 76.2 0)
 			(hide yes)
@@
 			)
 		)
-		(property "Lily_ID" "NO_ID"
+		(property "Lily_ID" "1914-10004"
 			(at 81.28 68.58 0)
 			(hide yes)
