File: test_projects/lib_test/integrated_circuits/voltage_regulators.kicad_sch (KiCad schematic)
At the start: 9 parts, among them U1022 REF3040, U1023 AP2120N-3.3, U1024 AZ1117C, U1025 AP62200, U1026 TPS5430, U1027 TPS82130, U1028 LM317, U1029 LM337, U1035 AP2205

Commit message: updated Lily IDs
Parts:
- U1022: Lily_ID NO_ID -> 1914-10027
- U1023: Lily_ID NO_ID -> 1914-10028
- U1024: Lily_ID NO_ID -> 1914-10031
- U1025: Lily_ID NO_ID -> 1914-10030
- U1026: Lily_ID NO_ID -> 1914-10034
- U1027: Lily_ID NO_ID -> 1914-10035
- U1028: Lily_ID NO_ID -> 1914-10032
- U1029: Lily_ID NO_ID -> 1914-10033
- U1035: Lily_ID NO_ID -> 1914-10029
Changed lines of the file:
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@@
 			)
 		)
-		(property "Lily_ID" "NO_ID"
+		(property "Lily_ID" "1914-10027"
 			(at 35.56 60.96 0)
 			(hide yes)
@@
 			)
 		)
-		(property "Lily_ID" "NO_ID"
+		(property "Lily_ID" "1914-10031"
 			(at 111.76 58.42 0)
 			(hide yes)
@@
 			)
 		)
-		(property "Lily_ID" "NO_ID"
+		(property "Lily_ID" "1914-10033"
 			(at 73.66 81.28 0)
 			(hide yes)
@@
 			)
 		)
-		(property "Lily_ID" "NO_ID"
+		(property "Lily_ID" "1914-10030"
 			(at 152.4 76.2 0)
 			(hide yes)
@@
 			)
 		)
-		(property "Lily_ID" "NO_ID"
+		(property "Lily_ID" "1914-10028"
 			(at 73.66 60.96 0)
 			(hide yes)
@@
 			)
 		)
-		(property "Lily_ID" "NO_ID"
+		(property "Lily_ID" "1914-10032"
 			(at 35.56 81.28 0)
 			(hide yes)
@@
 			)
 		)
-		(property "Lily_ID" "NO_ID"
+		(property "Lily_ID" "1914-10034"
 			(at 203.2 78.74 0)
 			(hide yes)
@@
 			)
 		)
-		(property "Lily_ID" "NO_ID"
+		(property "Lily_ID" "1914-10029"
 			(at 114.3 88.9 0)
 			(hide yes)
@@
 			)
 		)
-		(property "Lily_ID" "NO_ID"
+		(property "Lily_ID" "1914-10035"
 			(at 254 83.82 0)
 			(hide yes)
