File: test_projects/lib_test/integrated_circuits/opto_couplers.kicad_sch (KiCad schematic)
At the start: 1 part, among them U1036 MOC3023

Commit message: add triac
Parts:
- U1036: Lily_ID NO_ID -> 1914-10036
Changed lines of the file:
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@@
 			)
 		)
-		(property "Lily_ID" "NO_ID"
+		(property "Lily_ID" "1914-10036"
 			(at 49.53 67.31 0)
 			(hide yes)
