File: test_projects/lib_test/potentiometers/potentiometers.kicad_sch (KiCad schematic)
At the start: 5 parts, among them P1001 500R, P1002 2k, P1003 5k, P1004 1k

Commit message: updated Lily IDs
Parts:
- P1001: Lily_ID NO_ID -> 1919-10003
- P1002: Lily_ID NO_ID -> 1919-10002
- P1003: Lily_ID NO_ID -> 1919-10004
- P1004: Lily_ID NO_ID -> 1919-10001
Changed lines of the file:
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@@
 			)
 		)
-		(property "Lily_ID" "NO_ID"
+		(property "Lily_ID" "1919-10004"
 			(at 50.8 53.34 0)
 			(hide yes)
@@
 			)
 		)
-		(property "Lily_ID" "NO_ID"
+		(property "Lily_ID" "1919-10002"
 			(at 38.1 53.34 0)
 			(hide yes)
@@
 			)
 		)
-		(property "Lily_ID" "NO_ID"
+		(property "Lily_ID" "1919-10003"
 			(at 25.4 53.34 0)
 			(hide yes)
@@
 		(in_bom yes)
 		(on_board yes)
-		(in_pos_files no)
+		(in_pos_files yes)
 		(dnp no)
 		(property "Reference" "P1004"
@@
 			)
 		)
-		(property "Lily_ID" "NO_ID"
+		(property "Lily_ID" "1919-10001"
 			(at 25.4 66.04 0)
 			(hide yes)
