File: test_projects/lib_test/resistors/resistors.kicad_sch (KiCad schematic)
At the start: 172 parts

Commit message: updated Lily IDs
Parts:
- R1001: Lily_ID NO_ID -> 1913-11000
- R1002: Lily_ID NO_ID -> 1913-11100
- R1003: Lily_ID NO_ID -> 1913-11200
- R1004: Lily_ID NO_ID -> 1913-11300
- R1005: Lily_ID NO_ID -> 1913-11500
- R1006: Lily_ID NO_ID -> 1913-11600
- R1007: Lily_ID NO_ID -> 1913-11800
- R1008: Lily_ID NO_ID -> 1913-12000
- R1009: Lily_ID NO_ID -> 1913-12200
- R1010: Lily_ID NO_ID -> 1913-12400
- R1011: Lily_ID NO_ID -> 1913-12700
- R1012: Lily_ID NO_ID -> 1913-13000
- R1013: Lily_ID NO_ID -> 1913-13300
- R1014: Lily_ID NO_ID -> 1913-13600
- R1015: Lily_ID NO_ID -> 1913-13900
- R1016: Lily_ID NO_ID -> 1913-14300
- R1017: Lily_ID NO_ID -> 1913-14700
- R1018: Lily_ID NO_ID -> 1913-15100
- R1019: Lily_ID NO_ID -> 1913-15600
- R1020: Lily_ID NO_ID -> 1913-16200
- R1021: Lily_ID NO_ID -> 1913-16800
- R1022: Lily_ID NO_ID -> 1913-17500
- R1023: Lily_ID NO_ID -> 1913-18200
- R1024: Lily_ID NO_ID -> 1913-19100
- R1025: Lily_ID NO_ID -> 1913-11001
- R1026: Lily_ID NO_ID -> 1913-11101
- R1027: Lily_ID NO_ID -> 1913-11201
- R1028: Lily_ID NO_ID -> 1913-11301
- R1029: Lily_ID NO_ID -> 1913-11501
- R1030: Lily_ID NO_ID -> 1913-11601
- R1031: Lily_ID NO_ID -> 1913-11801
- R1032: Lily_ID NO_ID -> 1913-12001
- R1033: Lily_ID NO_ID -> 1913-12201
- R1034: Lily_ID NO_ID -> 1913-12401
- R1035: Lily_ID NO_ID -> 1913-12701
- R1036: Lily_ID NO_ID -> 1913-13001
- R1037: Lily_ID NO_ID -> 1913-13301
- R1038: Lily_ID NO_ID -> 1913-13601
- R1039: Lily_ID NO_ID -> 1913-13901
- R1040: Lily_ID NO_ID -> 1913-14301
- R1041: Lily_ID NO_ID -> 1913-14701
- R1042: Lily_ID NO_ID -> 1913-15101
- R1043: Lily_ID NO_ID -> 1913-15601
- R1044: Lily_ID NO_ID -> 1913-16201
- R1045: Lily_ID NO_ID -> 1913-16801
- R1046: Lily_ID NO_ID -> 1913-17501
- R1047: Lily_ID NO_ID -> 1913-18201
- R1048: Lily_ID NO_ID -> 1913-19101
- R1049: Lily_ID NO_ID -> 1913-11002
- R1050: Lily_ID NO_ID -> 1913-11102
- R1051: Lily_ID NO_ID -> 1913-11202
- R1052: Lily_ID NO_ID -> 1913-11302
- R1053: Lily_ID NO_ID -> 1913-11502
- R1054: Lily_ID NO_ID -> 1913-11602
- R1055: Lily_ID NO_ID -> 1913-11802
- R1056: Lily_ID NO_ID -> 1913-12002
- R1057: Lily_ID NO_ID -> 1913-12202
- R1058: Lily_ID NO_ID -> 1913-12402
- R1059: Lily_ID NO_ID -> 1913-12702
- R1060: Lily_ID NO_ID -> 1913-13002
- R1061: Lily_ID NO_ID -> 1913-13302
- R1062: Lily_ID NO_ID -> 1913-13602
- R1063: Lily_ID NO_ID -> 1913-13902
- R1064: Lily_ID NO_ID -> 1913-14302
- R1065: Lily_ID NO_ID -> 1913-14702
- R1066: Lily_ID NO_ID -> 1913-15102
- R1067: Lily_ID NO_ID -> 1913-15602
- R1068: Lily_ID NO_ID -> 1913-16202
- R1069: Lily_ID NO_ID -> 1913-16802
- R1070: Lily_ID NO_ID -> 1913-17502
- R1071: Lily_ID NO_ID -> 1913-18202
- R1072: Lily_ID NO_ID -> 1913-19102
- R1073: Lily_ID NO_ID -> 1913-11003
- R1074: Lily_ID NO_ID -> 1913-11103
- R1075: Lily_ID NO_ID -> 1913-11203
- R1076: Lily_ID NO_ID -> 1913-11303
- R1077: Lily_ID NO_ID -> 1913-11503
- R1078: Lily_ID NO_ID -> 1913-11603
- R1079: Lily_ID NO_ID -> 1913-11803
- R1080: Lily_ID NO_ID -> 1913-12003
- R1081: Lily_ID NO_ID -> 1913-12203
- R1082: Lily_ID NO_ID -> 1913-12403
- R1083: Lily_ID NO_ID -> 1913-12703
- R1084: Lily_ID NO_ID -> 1913-13003
- R1085: Lily_ID NO_ID -> 1913-13303
- R1086: Lily_ID NO_ID -> 1913-13603
- R1087: Lily_ID NO_ID -> 1913-13903
- R1088: Lily_ID NO_ID -> 1913-14303
- R1089: Lily_ID NO_ID -> 1913-14703
- R1090: Lily_ID NO_ID -> 1913-15103
- R1091: Lily_ID NO_ID -> 1913-15603
- R1092: Lily_ID NO_ID -> 1913-16203
- R1093: Lily_ID NO_ID -> 1913-16803
- R1094: Lily_ID NO_ID -> 1913-17503
- R1095: Lily_ID NO_ID -> 1913-18203
- R1096: Lily_ID NO_ID -> 1913-19103
- R1097: Lily_ID NO_ID -> 1913-11004
- R1098: Lily_ID NO_ID -> 1913-11104
- R1099: Lily_ID NO_ID -> 1913-11204
- R1100: Lily_ID NO_ID -> 1913-11304
- R1101: Lily_ID NO_ID -> 1913-11504
- R1102: Lily_ID NO_ID -> 1913-11604
- R1103: Lily_ID NO_ID -> 1913-11804
- R1104: Lily_ID NO_ID -> 1913-12004
- R1105: Lily_ID NO_ID -> 1913-12204
- R1106: Lily_ID NO_ID -> 1913-12404
- R1107: Lily_ID NO_ID -> 1913-12704
- R1108: Lily_ID NO_ID -> 1913-13004
- R1109: Lily_ID NO_ID -> 1913-13304
- R1110: Lily_ID NO_ID -> 1913-13604
- R1111: Lily_ID NO_ID -> 1913-13904
- R1112: Lily_ID NO_ID -> 1913-14304
- R1113: Lily_ID NO_ID -> 1913-14704
- R1114: Lily_ID NO_ID -> 1913-15104
- R1115: Lily_ID NO_ID -> 1913-15604
- R1116: Lily_ID NO_ID -> 1913-16204
- R1117: Lily_ID NO_ID -> 1913-16804
- R1118: Lily_ID NO_ID -> 1913-17504
- R1119: Lily_ID NO_ID -> 1913-18204
- R1120: Lily_ID NO_ID -> 1913-19104
- R1121: Lily_ID NO_ID -> 1913-11005
- R1122: Lily_ID NO_ID -> 1913-11105
- R1123: Lily_ID NO_ID -> 1913-11205
- R1124: Lily_ID NO_ID -> 1913-11305
- R1125: Lily_ID NO_ID -> 1913-11505
- R1126: Lily_ID NO_ID -> 1913-11605
- R1127: Lily_ID NO_ID -> 1913-11805
- R1128: Lily_ID NO_ID -> 1913-12005
- R1129: Lily_ID NO_ID -> 1913-12205
- R1130: Lily_ID NO_ID -> 1913-12405
- R1131: Lily_ID NO_ID -> 1913-12705
- R1132: Lily_ID NO_ID -> 1913-13005
- R1133: Lily_ID NO_ID -> 1913-13305
- R1134: Lily_ID NO_ID -> 1913-13605
- R1135: Lily_ID NO_ID -> 1913-13905
- R1136: Lily_ID NO_ID -> 1913-14305
- R1137: Lily_ID NO_ID -> 1913-14705
- R1138: Lily_ID NO_ID -> 1913-15105
- R1139: Lily_ID NO_ID -> 1913-15605
- R1140: Lily_ID NO_ID -> 1913-16205
- R1141: Lily_ID NO_ID -> 1913-16805
- R1142: Lily_ID NO_ID -> 1913-17505
- R1143: Lily_ID NO_ID -> 1913-18205
- R1144: Lily_ID NO_ID -> 1913-19105
- R1145: Lily_ID NO_ID -> 1913-11006
- R1146: Lily_ID NO_ID -> 1913-11106
- R1147: Lily_ID NO_ID -> 1913-11206
- R1148: Lily_ID NO_ID -> 1913-11306
- R1149: Lily_ID NO_ID -> 1913-11506
- R1150: Lily_ID NO_ID -> 1913-11606
- R1151: Lily_ID NO_ID -> 1913-11806
- R1152: Lily_ID NO_ID -> 1913-12006
- R1153: Lily_ID NO_ID -> 1913-12206
- R1154: Lily_ID NO_ID -> 1913-12406
- R1155: Lily_ID NO_ID -> 1913-12706
- R1156: Lily_ID NO_ID -> 1913-13006
- R1157: Lily_ID NO_ID -> 1913-13306
- R1158: Lily_ID NO_ID -> 1913-13606
- R1159: Lily_ID NO_ID -> 1913-13906
- R1160: Lily_ID NO_ID -> 1913-14306
- R1161: Lily_ID NO_ID -> 1913-14706
- R1162: Lily_ID NO_ID -> 1913-15106
- R1163: Lily_ID NO_ID -> 1913-15606
- R1164: Lily_ID NO_ID -> 1913-16206
- R1165: Lily_ID NO_ID -> 1913-16806
- R1166: Lily_ID NO_ID -> 1913-17506
- R1167: Lily_ID NO_ID -> 1913-18206
- R1168: Lily_ID NO_ID -> 1913-19106
- R1169: Lily_ID NO_ID -> 1913-10000
- R1170: Lily_ID NO_ID -> 1913-90001
- R1171: Lily_ID NO_ID -> 1913-90002
- R1172: Lily_ID NO_ID -> 1913-90003
