File: test_projects/lib_test/switches/switches.kicad_sch (KiCad schematic)
At the start: 2 parts

Commit message: updated Lily IDs
Parts:
- S1001: Lily_ID NO_ID -> 1920-10003
- S1002: Lily_ID NO_ID -> 1920-10002
Changed lines of the file:
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@@
 			)
 		)
-		(property "Lily_ID" "NO_ID"
+		(property "Lily_ID" "1920-10002"
 			(at 57.15 48.26 0)
 			(hide yes)
@@
 			)
 		)
-		(property "Lily_ID" "NO_ID"
+		(property "Lily_ID" "1920-10002"
 			(at 44.45 48.26 0)
 			(hide yes)
@@
 			)
 		)
-		(property "Lily_ID" "NO_ID"
+		(property "Lily_ID" "1920-10003"
 			(at 27.94 55.88 0)
 			(hide yes)
